Commit message: got codfather model to load; collada files not supported apparently

File: usv_sim/xacro/codfather.xacro (robot description, xacro)
@@ -21,5 +21,5 @@
 		<visual name="visual">
 			<geometry>
-				<mesh filename="package://usv_sim/meshes/codfather/deck_hull.dae" scale="1 1 1" />
+				<mesh filename="package://usv_sim/meshes/codfather/deck_hull_convex_hull.obj" scale="1 1 1" />
 			</geometry>
 			<origin rpy="0 0 0" xyz="0 0 1.4478" />
@@ -55,5 +55,5 @@
 		<visual name="ballast_visual">
 			<geometry>
-				<mesh filename="package://usv_sim/meshes/codfather/ballast.dae" scale="1 1 1" />
+				<mesh filename="package://usv_sim/meshes/codfather/ballast_convex_hull.obj" scale="1 1 1" />
 			</geometry>
 			<origin rpy="0 0 0" xyz="-0.225 0 0.0974" />
@@ -75,5 +75,5 @@
 		<visual name="mast_visual">
 			<geometry>
-				<mesh filename="package://usv_sim/meshes/codfather/mast.dae" scale="1 1 1" />
+				<mesh filename="package://usv_sim/meshes/codfather/MainAxle.obj" scale="1 1 1" />
 			</geometry>
 			<!-- <origin rpy="0 0 0" xyz="0 0 1.968" /> -->
@@ -104,5 +104,5 @@
 		<visual name="sail_visual">
 			<geometry>
-				<mesh filename="package://usv_sim/meshes/codfather/sail.dae" scale="1 1 1" />
+				<mesh filename="package://usv_sim/meshes/codfather/sail_alone_convex_hull.obj" scale="1 1 1" />
 			</geometry>
 			<origin rpy="0 0 3.1415926535897932" xyz="0 0 0.6726" />
@@ -127,5 +127,5 @@
 		<visual name="axle_visual">
 			<geometry>
-				<mesh filename="package://usv_sim/meshes/codfather/axle.dae" scale="1 1 1" />
+				<mesh filename="package://usv_sim/meshes/codfather/RudderAxle_convex_hull.obj" scale="1 1 1" />
 			</geometry>
 			<!-- <origin rpy="0 0 0" xyz="-0.894724 0 1.3970" /> -->
@@ -139,5 +139,5 @@
 		<visual name="rudder_visual">
 			<geometry>
-				<mesh filename="package://usv_sim/meshes/codfather/rudder.dae" scale="1 1 1" />
+				<mesh filename="package://usv_sim/meshes/codfather/rudder_convex_hull.obj" scale="1 1 1" />
 			</geometry>
 			<origin rpy="0 0 0" xyz="0 0 -0.0508" />

Commit message: Adding materials to codfather obj files

File: usv_sim/xacro/codfather.xacro (robot description, xacro)
@@ -15,5 +15,5 @@
 		<collision name="collision">
 			<geometry>
-				<mesh filename="package://usv_sim/meshes/codfather/deck_hull_convex_hull.obj" scale="1 1 1" />
+				<mesh filename="package://usv_sim/meshes/codfather/deck_hull_colored.obj" scale="1 1 1" />
 			</geometry>
 			<origin rpy="0 0 0" xyz="0 0 1.4478" />
@@ -21,5 +21,5 @@
 		<visual name="visual">
 			<geometry>
-				<mesh filename="package://usv_sim/meshes/codfather/deck_hull_convex_hull.obj" scale="1 1 1" />
+				<mesh filename="package://usv_sim/meshes/codfather/deck_hull_colored.obj" scale="1 1 1" />
 			</geometry>
 			<origin rpy="0 0 0" xyz="0 0 1.4478" />
@@ -35,5 +35,5 @@
 		<visual name="keel_visual">
 			<geometry>
-				<mesh filename="package://usv_sim/meshes/codfather/keel.obj" scale="1 1 1" />
+				<mesh filename="package://usv_sim/meshes/codfather/keel_colored.obj" scale="1 1 1" />
 			</geometry>
 			<origin rpy="0 0 0" xyz="-0.0762 0 0.7648" />
@@ -41,5 +41,5 @@
 		<collision name="keel_collision">
 			<geometry>
-				<mesh filename="package://usv_sim/meshes/codfather/keel.obj" scale="1 1 1" />
+				<mesh filename="package://usv_sim/meshes/codfather/keel_colored.obj" scale="1 1 1" />
 			</geometry>
 			<origin rpy="0 0 0" xyz="-0.0762 0 0.7648" />
@@ -55,5 +55,5 @@
 		<visual name="ballast_visual">
 			<geometry>
-				<mesh filename="package://usv_sim/meshes/codfather/ballast_convex_hull.obj" scale="1 1 1" />
+				<mesh filename="package://usv_sim/meshes/codfather/ballast_colored.obj" scale="1 1 1" />
 			</geometry>
 			<origin rpy="0 0 0" xyz="-0.225 0 0.0974" />
@@ -61,5 +61,5 @@
 		<collision name="ballast_collision">
 			<geometry>
-				<mesh filename="package://usv_sim/meshes/codfather/ballast_convex_hull.obj" scale="1 1 1" />
+				<mesh filename="package://usv_sim/meshes/codfather/ballast_colored.obj" scale="1 1 1" />
 			</geometry>
 			<origin rpy="0 0 0" xyz="-0.225 0 0.0974" />
@@ -75,5 +75,5 @@
 		<visual name="mast_visual">
 			<geometry>
-				<mesh filename="package://usv_sim/meshes/codfather/MainAxle.obj" scale="1 1 1" />
+				<mesh filename="package://usv_sim/meshes/codfather/mast_colored.obj" scale="1 1 1" />
 			</geometry>
 			<!-- <origin rpy="0 0 0" xyz="0 0 1.968" /> -->
@@ -82,5 +82,5 @@
 		<collision name="mast_collision">
 			<geometry>
-				<mesh filename="package://usv_sim/meshes/codfather/MainAxle.obj" scale="1 1 1" />
+				<mesh filename="package://usv_sim/meshes/codfather/mast_colored.obj" scale="1 1 1" />
 			</geometry>
 			<!-- <origin rpy="0 0 0" xyz="0 0 1.968" /> -->
@@ -97,5 +97,5 @@
 		<collision name="sail_collision">
 			<geometry>
-				<mesh filename="package://usv_sim/meshes/codfather/sail_alone_convex_hull.obj" scale="1 1 1" />
+				<mesh filename="package://usv_sim/meshes/codfather/sail_colored.obj" scale="1 1 1" />
 			</geometry>
 			<!-- <origin rpy="0 0 3.1415926535897932" xyz="0 0 2.1204" /> -->
@@ -104,5 +104,5 @@
 		<visual name="sail_visual">
 			<geometry>
-				<mesh filename="package://usv_sim/meshes/codfather/sail_alone_convex_hull.obj" scale="1 1 1" />
+				<mesh filename="package://usv_sim/meshes/codfather/sail_colored.obj" scale="1 1 1" />
 			</geometry>
 			<origin rpy="0 0 3.1415926535897932" xyz="0 0 0.6726" />
@@ -125,13 +125,12 @@
 			<inertia ixx="0.0015580802136752137" ixy="-1.7161266666666664e-05" iyy="0.0017239371367521368" ixz="0.00010010581196581196" iyz="1.0223873504273504e-05" izz="0.0001771534829059829" />
 		</inertial>
-		<visual name="axle_visual">
+		<!-- <visual name="axle_visual">
 			<geometry>
 				<mesh filename="package://usv_sim/meshes/codfather/RudderAxle_convex_hull.obj" scale="1 1 1" />
 			</geometry>
-			<!-- <origin rpy="0 0 0" xyz="-0.894724 0 1.3970" /> -->
-		</visual>
+		</visual> -->
 		<collision name="rudder_collision">
 			<geometry>
-				<mesh filename="package://usv_sim/meshes/codfather/rudder_convex_hull.obj" scale="1 1 1" />
+				<mesh filename="package://usv_sim/meshes/codfather/rudder_colored.obj" scale="1 1 1" />
 			</geometry>
 			<origin rpy="0 0 0" xyz="0 0 -0.0508" />
@@ -139,5 +138,5 @@
 		<visual name="rudder_visual">
 			<geometry>
-				<mesh filename="package://usv_sim/meshes/codfather/rudder_convex_hull.obj" scale="1 1 1" />
+				<mesh filename="package://usv_sim/meshes/codfather/rudder_colored.obj" scale="1 1 1" />
 			</geometry>
 			<origin rpy="0 0 0" xyz="0 0 -0.0508" />
