Commit message: Codfather visuals added

File: usv_sim/xacro/boat_subdivided4.xacro (robot description, xacro)
@@ -1,438 +1,429 @@
 <?xml version="1.0"?>
 <xacro xmlns:xacro="http://www.ros.org/wiki/xacro">
-    <xacro:property name="PI" value="3.1415926535897931"/>
-    <!-- Body properties -->
-    <xacro:property name="front_body_mass" value="5"/>
-    <xacro:property name="back_body_mass" value="5"/>
-    <xacro:property name="middle_body_mass" value="5"/>
-    <xacro:property name="rear_body_mass" value="5"/>
-    <xacro:property name="front_body_mass" value="2"/>
-    <xacro:property name="back_water_displaced_mass" value="40"/>
-    <xacro:property name="middle_water_displaced_mass" value="40"/>
-    <xacro:property name="front_water_displaced_mass" value="25"/>
-    <xacro:property name="scale" value="0.3"/>
-    <xacro:property name="bl1" value=".1" />
-    <xacro:property name="bl2" value=".1" />
-    <xacro:arg name="windType" default="global" />
-    <xacro:arg name="waterType" default="global" />
-    <xacro:property name="windType" value="$(arg windType)" />
-    <xacro:property name="waterType" value="$(arg waterType)" />
-    <link name="base_link">
-        <visual>
-          <origin rpy="0 0 0" xyz="0 0 0"/>
-          <geometry>
-            <mesh filename="package://usv_sim/meshes/simpleHull3/base_link.dae" scale="${scale} ${scale} ${scale}"/>
-          </geometry>
-        </visual>
-        <collision>
-          <origin rpy="0 0 0" xyz="0 0 0"/>
-          <geometry>
-            <mesh filename="package://usv_sim/meshes/simpleHull3/base_link.dae" scale="${scale} ${scale} ${scale}"/>
-          </geometry>
-        </collision>
-        <inertial>
-            <origin rpy="0 0 0" xyz="${0.35*scale} ${0.44*scale} ${-0.2*scale}"/>
-          <mass value="${middle_body_mass}"/>
-          <inertia ixx="0.1" ixy="0.0" ixz="0.0" iyy="1.4" iyz="0.0" izz="1.4"/>
-        </inertial>
-        <buoyancy>
-			<compensation>${middle_water_displaced_mass/middle_body_mass}</compensation>
-			<origin xyz="${0.35*scale} ${0.44*scale} ${-0.15*scale}"/>
-			<limit radius="0.1"/>
-			<damping rpy="20 20 20" xyz="20 40 50"/>
-         	<windVelocity>${windType}</windVelocity>
-			<frontal_area>0.0</frontal_area>
-			<lateral_area>0.06</lateral_area>
-			<lateral_length>1.2</lateral_length>
-	  		<waterVelocity>${waterType}</waterVelocity>
-        </buoyancy>
+  <xacro:property name="PI" value="3.1415926535897931" />
+  <!-- Body properties -->
+  <xacro:property name="front_body_mass" value="5" />
+  <xacro:property name="back_body_mass" value="5" />
+  <xacro:property name="middle_body_mass" value="5" />
+  <xacro:property name="rear_body_mass" value="5" />
+  <xacro:property name="front_body_mass" value="2" />
+  <xacro:property name="back_water_displaced_mass" value="40" />
+  <xacro:property name="middle_water_displaced_mass" value="40" />
+  <xacro:property name="front_water_displaced_mass" value="25" />
+  <xacro:property name="scale" value="0.3" />
+  <xacro:property name="bl1" value=".1" />
+  <xacro:property name="bl2" value=".1" />
+  <xacro:arg name="windType" default="global" />
+  <xacro:arg name="waterType" default="global" />
+  <xacro:property name="windType" value="$(arg windType)" />
+  <xacro:property name="waterType" value="$(arg waterType)" />
+  <link name="base_link">
+    <!-- <visual>
+      <origin rpy="0 0 0" xyz="0 0 0" />
+      <geometry>
+        <mesh filename="package://usv_sim/meshes/simpleHull3/base_link.dae" scale="${scale} ${scale} ${scale}" />
+      </geometry>
+    </visual> -->
+    <visual>
+      <origin rpy="0 0 0" xyz="0.3 0 -0.15" />
+      <geometry>
+        <mesh filename="package://usv_sim/meshes/codfather/deck_hull_colored.obj" scale="1 1 1" />
+      </geometry>
+    </visual>
+    <collision>
+      <origin rpy="0 0 0" xyz="0 0 0" />
+      <geometry>
+        <mesh filename="package://usv_sim/meshes/simpleHull3/base_link.dae" scale="${scale} ${scale} ${scale}" />
+      </geometry>
+    </collision>
+    <inertial>
+      <origin rpy="0 0 0" xyz="${0.35*scale} ${0.44*scale} ${-0.2*scale}" />
+      <mass value="${middle_body_mass}" />
+      <inertia ixx="0.1" ixy="0.0" ixz="0.0" iyy="1.4" iyz="0.0" izz="1.4" />
+    </inertial>
+    <buoyancy>
+      <compensation>${middle_water_displaced_mass/middle_body_mass}</compensation>
+      <origin xyz="${0.35*scale} ${0.44*scale} ${-0.15*scale}" />
+      <limit radius="0.1" />
+      <damping rpy="20 20 20" xyz="20 40 50" />
+      <windVelocity>${windType}</windVelocity>
+      <frontal_area>0.0</frontal_area>
+      <lateral_area>0.06</lateral_area>
+      <lateral_length>1.2</lateral_length>
+      <waterVelocity>${waterType}</waterVelocity>
+    </buoyancy>
+  </link>
+  <link name="center_r_link">
+    <!-- <visual>
+      <origin rpy="0 0 0" xyz="0 0 ${0*scale}" />
+      <geometry>
+        <mesh filename="package://usv_sim/meshes/simpleHull3/centerRight.dae" scale="${scale} ${scale} ${scale}" />
+      </geometry>
+    </visual> -->
+    <collision>
+      <origin rpy="0 0 0" xyz="0 0 ${0*scale}" />
+      <geometry>
+        <mesh filename="package://usv_sim/meshes/simpleHull3/centerRight.dae" scale="${scale} ${scale} ${scale}" />
+      </geometry>
+    </collision>
+    <inertial>
+      <origin rpy="0 0 0" xyz="${0.35*scale} ${-0.44*scale} ${-0.2*scale}" />
+      <mass value="${middle_body_mass}" />
+      <inertia ixx="0.1" ixy="0.0" ixz="0.0" iyy="1.4" iyz="0.0" izz="1.4" />
+    </inertial>
+    <buoyancy>
+      <compensation>${middle_water_displaced_mass/middle_body_mass}</compensation>
+      <origin xyz="${0.35*scale} ${-0.44*scale} ${-0.15*scale}" />
+      <limit radius="0.1" />
+      <damping rpy="20 20 20" xyz="20 40 50" />
+      <windVelocity>${windType}</windVelocity>
+      <frontal_area>0.0</frontal_area>
+      <lateral_area>0.06</lateral_area>
+      <lateral_length>1.2</lateral_length>
+      <waterVelocity>${waterType}</waterVelocity>
+    </buoyancy>
+  </link>
+  <joint name="center_r_joint" type="revolute">
+    <parent link="base_link" />
+    <child link="center_r_link" />
+    <origin rpy="0 0 0" xyz="0 0 0" />
+    <limit effort="50" velocity="5" lower="0" upper="0" />
+    <dynamics damping="1.0" />
+    <axis xyz="1 0 0" />
+  </joint>
+  <link name="back_l_link">
+    <!-- <visual>
+      <origin rpy="0 0 0" xyz="0 0 0" />
+      <geometry>
+        <mesh filename="package://usv_sim/meshes/simpleHull3/backLeft.dae" scale="${scale} ${scale} ${scale}" />
+      </geometry>
+    </visual> -->
+    <collision>
+      <origin rpy="0 0 0" xyz="0 0 0" />
+      <geometry>
+        <mesh filename="package://usv_sim/meshes/simpleHull3/backLeft.dae" scale="${scale} ${scale} ${scale}" />
+      </geometry>
+    </collision>
+    <inertial>
+      <origin rpy="0 0 0" xyz="${-0.6*scale} 0 ${-0.2*scale}" />
+      <mass value="${back_body_mass}" />
+      <inertia ixx="0.1" ixy="0.0" ixz="0.0" iyy="1.4" iyz="0.0" izz="1.4" />
+    </inertial>
+    <buoyancy>
+      <compensation>${back_water_displaced_mass/back_body_mass}</compensation>
+      <origin xyz="${-0.6*scale} 0 ${-0.15*scale}" />
+      <limit radius="0.1" />
+      <damping rpy="20 20 20" xyz="20 40 50" />
+      <windVelocity>${windType}</windVelocity>
+      <frontal_area>0.04</frontal_area>
+      <lateral_area>0.06</lateral_area>
+      <lateral_length>1.2</lateral_length>
+      <waterVelocity>${waterType}</waterVelocity>
+    </buoyancy>
+  </link>
+  <joint name="back_l_joint" type="revolute">
+    <parent link="base_link" />
+    <child link="back_l_link" />
+    <origin rpy="0 0 0" xyz="${-0.5*scale} ${0.39*scale} 0" />
+    <limit effort="50" velocity="5" lower="0" upper="0" />
+    <dynamics damping="1.0" />
+    <axis xyz="1 0 0" />
+  </joint>
+  <link name="back_r_link">
+    <!-- <visual>
+      <origin rpy="0 0 0" xyz="0 0 0" />
+      <geometry>
+        <mesh filename="package://usv_sim/meshes/simpleHull3/backRight.dae" scale="${scale} ${scale} ${scale}" />
+      </geometry>
+    </visual> -->
+    <collision>
+      <origin rpy="0 0 0" xyz="0 0 0" />
+      <geometry>
+        <mesh filename="package://usv_sim/meshes/simpleHull3/backRight.dae" scale="${scale} ${scale} ${scale}" />
+      </geometry>
+    </collision>
+    <inertial>
+      <origin rpy="0 0 0" xyz="${-0.6*scale} 0 ${-0.2*scale}" />
+      <mass value="${back_body_mass}" />
+      <inertia ixx="0.1" ixy="0.0" ixz="0.0" iyy="1.4" iyz="0.0" izz="1.4" />
+    </inertial>
+    <buoyancy>
+      <compensation>${back_water_displaced_mass/back_body_mass}</compensation>
+      <origin xyz="${-0.6*scale} 0 ${-0.15*scale}" />
+      <limit radius="0.1" />
+      <damping rpy="20 20 20" xyz="20 40 50" />
+      <windVelocity>${windType}</windVelocity>
+      <frontal_area>0.04</frontal_area>
+      <lateral_area>0.06</lateral_area>
+      <lateral_length>1.2</lateral_length>
+      <waterVelocity>${waterType}</waterVelocity>
+    </buoyancy>
+  </link>
+  <joint name="back_r_joint" type="revolute">
+    <parent link="base_link" />
+    <child link="back_r_link" />
+    <origin rpy="0 0 0" xyz="${-0.5*scale} ${-0.39*scale} 0" />
+    <limit effort="50" velocity="5" lower="0" upper="0" />
+    <dynamics damping="1.0" />
+    <axis xyz="1 0 0" />
+  </joint>
+  <link name="front_l_link">
+    <!-- <visual>
+      <origin rpy="0 0 0" xyz="0 0 0" />
+      <geometry>
+        <mesh filename="package://usv_sim/meshes/simpleHull3/frontLeft.dae" scale="${scale} ${scale} ${scale}" />
+      </geometry>
+    </visual> -->
+    <collision>
+      <origin rpy="0 0 0" xyz="0 0 0" />
+      <geometry>
+        <mesh filename="package://usv_sim/meshes/simpleHull3/frontLeft.dae" scale="${scale} ${scale} ${scale}" />
+      </geometry>
+    </collision>
+    <inertial>
+      <origin rpy="0 0 0" xyz="${0.4*scale} 0 ${-0.1*scale}" />
+      <mass value="${front_body_mass}" />
+      <inertia ixx="0.1" ixy="0.0" ixz="0.0" iyy="1.4" iyz="0.0" izz="1.4" />
+    </inertial>
+    <buoyancy>
+      <compensation>${front_water_displaced_mass/front_body_mass}</compensation>
+      <origin xyz="${0.4*scale} 0 ${-0.05*scale}" />
+      <limit radius="0.1" />
+      <damping rpy="20 20 20" xyz="20 40 50" />
+      <windVelocity>${windType}</windVelocity>
+      <frontal_area>0.04</frontal_area>
+      <lateral_area>0.06</lateral_area>
+      <lateral_length>1.2</lateral_length>
+      <waterVelocity>${waterType}</waterVelocity>
+    </buoyancy>
+  </link>
+  <joint name="front_l_joint" type="revolute">
+    <parent link="base_link" />
+    <child link="front_l_link" />
+    <origin rpy="0 0 0" xyz="${1.3*scale} ${0.2*scale} 0" />
+    <limit effort="50" velocity="5" lower="0" upper="0" />
+    <dynamics damping="1.0" />
+    <axis xyz="1 0 0" />
+  </joint>
+  <link name="front_r_link">
+    <!-- <visual>
+      <origin rpy="0 0 0" xyz="0 0 0" />
+      <geometry>
+        <mesh filename="package://usv_sim/meshes/simpleHull3/frontRight.dae" scale="${scale} ${scale} ${scale}" />
+      </geometry>
+    </visual> -->
+    <collision>
+      <origin rpy="0 0 0" xyz="${0*scale} ${0*scale} 0" />
+      <geometry>
+        <mesh filename="package://usv_sim/meshes/simpleHull3/frontRight.dae" scale="${scale} ${scale} ${scale}" />
+      </geometry>
+    </collision>
+    <inertial>
+      <origin rpy="0 0 0" xyz="${0.4*scale} 0 ${-0.1*scale}" />
+      <mass value="${front_body_mass}" />
+      <inertia ixx="0.1" ixy="0.0" ixz="0.0" iyy="1.4" iyz="0.0" izz="1.4" />
+    </inertial>
+    <buoyancy>
+      <compensation>${front_water_displaced_mass/front_body_mass}</compensation>
+      <origin xyz="${0.4*scale} 0 ${-0.05*scale}" />
+      <limit radius="0.1" />
+      <damping rpy="20 20 20" xyz="20 40 50" />
+      <windVelocity>${windType}</windVelocity>
+      <waterVelocity>${waterType}</waterVelocity>
+    </buoyancy>
+  </link>
+  <joint name="front_r_joint" type="revolute">
+    <parent link="base_link" />
+    <child link="front_r_link" />
+    <origin rpy="0 0 0" xyz="${1.3*scale} ${-0.2*scale} 0" />
+    <limit effort="50" velocity="5" lower="0" upper="0" />
+    <dynamics damping="1.0" />
+    <axis xyz="1 0 0" />
+  </joint>
+  <!-- Thruster link -->
+  <xacro:macro name="thruster_link" params="name xyz rpy rotationAxis effort:=50 velocity:=5 lowerLimit upperLimit parentLink:=back_r_link">
+    <joint name="${name}_joint" type="revolute">
+      <parent link="${parentLink}" />
+      <child link="${name}" />
+      <origin rpy="${rpy}" xyz="${xyz}" />
+      <dynamics damping="10.0" />
+      <axis xyz="${rotationAxis}" />
+      <limit effort="${effort}" velocity="${velocity}" lower="${lowerLimit}" upper="${upperLimit}" />
+    </joint>
+    <link name="${name}">
+      <buoyancy>
+        <compensation>0.8</compensation>
+        <waterVelocity>${waterType}</waterVelocity>
+      </buoyancy>
+      <collision>
+        <origin xyz="${-0.15*scale} 0 ${0*scale}" rpy="0 0 0" />
+        <geometry>
+          <mesh filename="package://usv_sim/meshes/simpleHull3/thruster.dae" scale="${scale} ${scale} ${scale}" />
+        </geometry>
+      </collision>
+      <visual name="${name}">
+        <origin xyz="${-0.15*scale} 0 ${0*scale}" rpy="0 0 0" />
+        <geometry>
+          <mesh filename="package://usv_sim/meshes/simpleHull3/thruster.dae" scale="${scale} ${scale} ${scale}" />
+        </geometry>
+        <material name="black">
+          <color rgba="255 255 255 1" />
+        </material>
+      </visual>
+      <inertial>
+        <mass value="5" />
+        <origin xyz="${-0.2*scale} 0 ${0.3*scale}" rpy="0 0 0" />
+        <inertia ixx=".1" ixy="0.0" ixz="0.0" iyy=".1" iyz="0.0" izz=".1" />
+      </inertial>
     </link>
-    <link name="center_r_link">
-    	<visual>
-          <origin rpy="0 0 0"  xyz="0 0 ${0*scale}"/>
-          <geometry>
-            <mesh filename="package://usv_sim/meshes/simpleHull3/centerRight.dae" scale="${scale} ${scale} ${scale}"/>
-          </geometry>
-        </visual>
-        <collision>
-          <origin rpy="0 0 0"  xyz="0 0 ${0*scale}"/>
-          <geometry>
-           	<mesh filename="package://usv_sim/meshes/simpleHull3/centerRight.dae" scale="${scale} ${scale} ${scale}"/>
-          </geometry>
-        </collision>
-        <inertial>
-            <origin rpy="0 0 0" xyz="${0.35*scale} ${-0.44*scale} ${-0.2*scale}"/>
-          <mass value="${middle_body_mass}"/>
-          <inertia ixx="0.1" ixy="0.0" ixz="0.0" iyy="1.4" iyz="0.0" izz="1.4"/>
-        </inertial>
-        <buoyancy>
-          <compensation>${middle_water_displaced_mass/middle_body_mass}</compensation>
-          <origin xyz="${0.35*scale} ${-0.44*scale} ${-0.15*scale}"/>
-          <limit radius="0.1"/>
-          <damping rpy="20 20 20" xyz="20 40 50"/>
-			<windVelocity>${windType}</windVelocity>
-			<frontal_area>0.0</frontal_area>
-			<lateral_area>0.06</lateral_area>
-			<lateral_length>1.2</lateral_length>
-	  <waterVelocity>${waterType}</waterVelocity>
-        </buoyancy>
+    <gazebo reference="${name}">
+      <material>Gazebo/Black</material>
+    </gazebo>
+  </xacro:macro>
+  <xacro:macro name="thruster_dummy_link" params="name xyz rpy">
+    <joint name="${name}" type="fixed">
+      <parent link="base_link" />
+      <child link="${name}" />
+      <origin rpy="${rpy}" xyz="${xyz}" />
+    </joint>
+    <link name="${name}" />
+  </xacro:macro>
+  <!-- Thruster link -->
+  <xacro:macro name="airthruster_link" params="name xyz rpy rotationAxis effort:=100 velocity:=20 lowerLimit upperLimit parentLink:=back_r_link">
+    <joint name="${name}_joint" type="revolute">
+      <parent link="${parentLink}" />
+      <child link="${name}" />
+      <origin rpy="${rpy}" xyz="${xyz}" />
+      <dynamics damping="10.0" />
+      <axis xyz="${rotationAxis}" />
+      <limit effort="${effort}" velocity="${velocity}" lower="${lowerLimit}" upper="${upperLimit}" />
+    </joint>
+    <link name="${name}">
+      <buoyancy>
+        <compensation>1.0</compensation>
+        <waterVelocity>${waterType}</waterVelocity>
+      </buoyancy>
+      <collision>
+        <origin xyz="0 0 0" rpy="0 0 0" />
+        <geometry>
+          <box size="${bl1} ${bl1} ${bl2}" />
+        </geometry>
+      </collision>
+      <visual name="${name}">
+        <origin xyz="0 0 0" rpy="0 0 0" />
+        <geometry>
+          <mesh filename="package://usv_sim/meshes/simpleHull3/airPropeller.dae" scale="${scale} ${scale} ${scale}" />
+        </geometry>
+      </visual>
+      <inertial>
+        <mass value=".1" />
+        <inertia ixx=".1" ixy="0.0" ixz="0.0" iyy=".1" iyz="0.0" izz=".1" />
+      </inertial>
     </link>
-    <joint name="center_r_joint" type="revolute">
-        <parent link="base_link"/>
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
File: usv_sim/xacro/codfather.xacro (robot description, xacro)
@@ -1,4 +1,8 @@
 <?xml version="1.0"?>
 <robot name="codfather" xmlns:xacro="http://www.ros.org/wiki/xacro">
+	<xacro:property name="body_mass" value="8" />
+	<!-- TODO figure out what this should be, I have no idea -->
+	<xacro:property name="body_water_displaced_mass" value="100" />
+	<xacro:property name="scale" value="1" />
 	<xacro:arg name="windType" default="global" />
 	<xacro:arg name="waterType" default="global" />
@@ -25,4 +29,15 @@
 			<origin rpy="0 0 0" xyz="0 0 1.4478" />
 		</visual>
+		<buoyancy>
+			<compensation>${body_water_displaced_mass/body_mass}</compensation>
+			<origin xyz="${0.35*scale} ${0.44*scale} ${-0.15*scale}" />
+			<limit radius="0.1" />
+			<damping rpy="20 20 20" xyz="20 40 50" />
+			<windVelocity>${windType}</windVelocity>
+			<frontal_area>0.04</frontal_area>
+			<lateral_area>0.06</lateral_area>
+			<lateral_length>1.2</lateral_length>
+			<waterVelocity>${waterType}</waterVelocity>
+		</buoyancy>
 	</link>
 	<link name="keel">
