Commit message: Codfather visuals added

File: usv_sim/xacro/sailboat.xacro (robot description, xacro)
@@ -1,135 +1,123 @@
 <?xml version="1.0"?>
 <robot name="sailboat" xmlns:xacro="http://www.ros.org/wiki/xacro">
-    <xacro:arg name="windType" default="global" />
-    <xacro:arg name="waterType" default="global" />
-    <xacro:property name="windType" value="$(arg windType)" />
-    <xacro:property name="waterType" value="$(arg waterType)" />
-    <xacro:property name="windType" value="global"/>
-    <xacro:include filename="$(find usv_sim)/xacro/boat_subdivided4.xacro" />
-    <xacro:rudder_xacro/>
-    <!-- Defining sail model -->
-    <link name="sail">
+	<xacro:arg name="windType" default="global" />
+	<xacro:arg name="waterType" default="global" />
+	<xacro:property name="windType" value="$(arg windType)" />
+	<xacro:property name="waterType" value="$(arg waterType)" />
+	<xacro:property name="windType" value="global" />
+	<xacro:include filename="$(find usv_sim)/xacro/boat_subdivided4.xacro" />
+	<xacro:rudder_xacro />
+	<!-- Defining sail model -->
+	<link name="sail">
 		<inertial>
-		    	<origin rpy="0 0 0" xyz="-0.3 0 0.4"/>
+			<origin rpy="0 0 0" xyz="-0.3 0 0.4" />
 			<mass value="1" />
-			<inertia
-			  ixx="0.4708"
-			  ixy="0.0"
-			  iyy="0.5208"
-			  ixz="0.0"
-			  iyz="0.0"
-			  izz="0.0508"/>
+			<inertia ixx="0.4708" ixy="0.0" iyy="0.5208" ixz="0.0" iyz="0.0" izz="0.0508" />
 		</inertial>
-	    <collision name="collision">
-            <geometry>
-              <mesh filename="package://usv_sim/meshes/simpleHull3/sail.dae" scale="0.5 0.5 0.5"/>
-            </geometry>
-            <origin rpy="0 0 0" xyz="0 0 0"/>
-	    </collision>
-	    <visual name="visual">
-            <geometry>
-              <mesh filename="package://usv_sim/meshes/simpleHull3/sail.dae" scale="0.5 0.5 0.5"/>
-            </geometry>
-            <origin rpy="0 0 0" xyz="0 0 0"/>
-	    </visual>
-    </link>
-    <joint name="sail_joint" type="revolute">
-        <parent link="base_link"/>
-        <child link="sail"/>
-        <origin rpy="0 0 0" xyz="0.2 0 0.1"/>
-        <dynamics damping="1.0"/>
-        <axis xyz="0 0 1"/>
-        <limit effort="100" velocity="70" lower="-${PI}" upper="${PI}" />
-    </joint>
-    <link name="keel">
-	<inertial>
-		<mass value="30" />
-		<inertia
-		  ixx="0.4708"
-		  ixy="0.0"
-		  iyy="0.5208"
-		  ixz="0.0"
-		  iyz="0.0"
-		  izz="0.0508"/>
-	</inertial>
-	<collision name="collision">
-		<geometry>
-			<box size="0.25 0.02 0.5" />
-		</geometry>
-		<origin rpy="0 0 0" xyz="0 0 0"/>
-	</collision>
-	<visual name="visual">
-		<geometry>
-			<mesh filename="package://usv_sim/meshes/simpleHull3/box.dae" scale="0.25 0.02 0.5"/>
-		</geometry>
-		<origin rpy="0 0 0" xyz="0 0 0"/>
-	</visual>
-</link>
-    <joint name="keel_joint" type="revolute">
-        <parent link="base_link"/>
-        <child link="keel"/>
-        <origin rpy="0 0 0" xyz="0 0 -0.35"/>
-        <dynamics damping="1.0"/>
-        <axis xyz="0 0 1"/>
-        <limit effort="30" velocity="5" lower="0" upper="0" />
-    </joint>
-    <!-- Plugin list -->
-  <gazebo>
-	<plugin name="usv_sail_plugin" filename="libfoil_dynamics_plugin.so">
-		<link_type>sail</link_type>
-		<a0>0</a0>
-		<cla>3.0</cla>
-		<cda>3.0</cda>
-		<cma>-1.8</cma>
-		<alpha_stall>0.785</alpha_stall>
-		<cla_stall>-3.85</cla_stall>
-		<cda_stall>-0.9233984055</cda_stall>
-		<cma_stall>0</cma_stall>
-		<cp>0 0 0</cp>
-		<joint_name>sail_joint</joint_name>
-		<area>1.44</area>
-		<fluid_density>1.2041</fluid_density>
-		<forward>-1 0 0</forward>
-		<upward>0 1 0</upward>
-		<link_name>sail</link_name>
-		<fluidVelocity>${windType}</fluidVelocity>
-      </plugin>
-      <plugin name="usv_sail_plugin" filename="libfoil_dynamics_plugin.so">
-		  <link_type>keel</link_type>
-		  <a0>0</a0>
-		  <cla>10.0</cla>
-		  <cda>8.0</cda>
-		  <alpha_stall>0.785</alpha_stall>
-		  <cla_stall>-10.0</cla_stall>
-		  <cda_stall>-5.0</cda_stall>
-		  <cp>0 0 0</cp>
-		  <area>1.0</area>
-		  <fluid_density>1000</fluid_density>
-		  <forward>1 0 0</forward>
-		  <upward>0 1 0</upward>
-		  <link_name>keel</link_name>
-		  <fluidVelocity>${waterType}</fluidVelocity>
-    </plugin>
-    <plugin name="usv_sail_plugin" filename="libfoil_dynamics_plugin.so">
-		<link_type>rudder</link_type>
-		<a0>0</a0>
-		<cla>0.8</cla>
-		<cda>0.3</cda>
-		<alpha_stall>0.785</alpha_stall>
-		<cla_stall>-0.85</cla_stall>
-		<cda_stall>-0.3233984055</cda_stall>
-		<cp>0 0 0</cp>
-		<area>1</area>
-		<fluid_density>1000</fluid_density>
-		<forward>1 0 0</forward>
-		<upward>0 1 0</upward>
-		<link_name>rudder</link_name>
-		<fluidVelocity>${waterType}</fluidVelocity>
-      </plugin>
-      <plugin name="freefloating_gazebo_control" filename="libfreefloating_gazebo_control.so">
-          <switchService>switch</switchService>
-          <updateRate>100</updateRate>
-          <link>base_link</link>
-      </plugin>
-  </gazebo>
+		<collision name="collision">
+			<geometry>
+				<mesh filename="package://usv_sim/meshes/simpleHull3/sail.dae" scale="0.5 0.5 0.5" />
+			</geometry>
+			<origin rpy="0 0 0" xyz="0 0 0" />
+		</collision>
+		<visual name="visual">
+			<geometry>
+				<mesh filename="package://usv_sim/meshes/codfather/sail_assem.obj" scale="1 1 1" />
+			</geometry>
+			<origin rpy="0 0 0" xyz="0 0 0.35" />
+		</visual>
+	</link>
+	<joint name="sail_joint" type="revolute">
+		<parent link="base_link" />
+		<child link="sail" />
+		<origin rpy="0 0 0" xyz="0.2 0 0.1" />
+		<dynamics damping="1.0" />
+		<axis xyz="0 0 1" />
+		<limit effort="100" velocity="70" lower="-${PI}" upper="${PI}" />
+	</joint>
+	<link name="keel">
+		<inertial>
+			<mass value="30" />
+			<inertia ixx="0.4708" ixy="0.0" iyy="0.5208" ixz="0.0" iyz="0.0" izz="0.0508" />
+		</inertial>
+		<collision name="collision">
+			<geometry>
+				<box size="0.25 0.02 0.5" />
+			</geometry>
+			<origin rpy="0 0 0" xyz="0 0 0" />
+		</collision>
+		<visual name="visual">
+			<geometry>
+				<mesh filename="package://usv_sim/meshes/codfather/keel_assem.obj" scale="0.25 0.02 0.5" />
+			</geometry>
+			<origin rpy="0 0 0" xyz="0.1 0 -0.2" />
+		</visual>
+	</link>
+	<joint name="keel_joint" type="revolute">
+		<parent link="base_link" />
+		<child link="keel" />
+		<origin rpy="0 0 0" xyz="0 0 -0.35" />
+		<dynamics damping="1.0" />
+		<axis xyz="0 0 1" />
+		<limit effort="30" velocity="5" lower="0" upper="0" />
+	</joint>
+	<!-- Plugin list -->
+	<gazebo>
+		<plugin name="usv_sail_plugin" filename="libfoil_dynamics_plugin.so">
+			<link_type>sail</link_type>
+			<a0>0</a0>
+			<cla>3.0</cla>
+			<cda>3.0</cda>
+			<cma>-1.8</cma>
+			<alpha_stall>0.785</alpha_stall>
+			<cla_stall>-3.85</cla_stall>
+			<cda_stall>-0.9233984055</cda_stall>
+			<cma_stall>0</cma_stall>
+			<cp>0 0 0</cp>
+			<joint_name>sail_joint</joint_name>
+			<area>1.44</area>
+			<fluid_density>1.2041</fluid_density>
+			<forward>-1 0 0</forward>
+			<upward>0 1 0</upward>
+			<link_name>sail</link_name>
+			<fluidVelocity>${windType}</fluidVelocity>
+		</plugin>
+		<plugin name="usv_sail_plugin" filename="libfoil_dynamics_plugin.so">
+			<link_type>keel</link_type>
+			<a0>0</a0>
+			<cla>10.0</cla>
+			<cda>8.0</cda>
+			<alpha_stall>0.785</alpha_stall>
+			<cla_stall>-10.0</cla_stall>
+			<cda_stall>-5.0</cda_stall>
+			<cp>0 0 0</cp>
+			<area>1.0</area>
+			<fluid_density>1000</fluid_density>
+			<forward>1 0 0</forward>
+			<upward>0 1 0</upward>
+			<link_name>keel</link_name>
+			<fluidVelocity>${waterType}</fluidVelocity>
+		</plugin>
+		<plugin name="usv_sail_plugin" filename="libfoil_dynamics_plugin.so">
+			<link_type>rudder</link_type>
+			<a0>0</a0>
+			<cla>0.8</cla>
+			<cda>0.3</cda>
+			<alpha_stall>0.785</alpha_stall>
+			<cla_stall>-0.85</cla_stall>
+			<cda_stall>-0.3233984055</cda_stall>
+			<cp>0 0 0</cp>
+			<area>1</area>
+			<fluid_density>1000</fluid_density>
+			<forward>1 0 0</forward>
+			<upward>0 1 0</upward>
+			<link_name>rudder</link_name>
+			<fluidVelocity>${waterType}</fluidVelocity>
+		</plugin>
+		<plugin name="freefloating_gazebo_control" filename="libfreefloating_gazebo_control.so">
+			<switchService>switch</switchService>
+			<updateRate>100</updateRate>
+			<link>base_link</link>
+		</plugin>
+	</gazebo>
 </robot>
