Commit message: Changing buoys

File: usv_sim/xacro/buoy.xacro (robot description, xacro)
@@ -3,28 +3,28 @@
   <link name="link">
     <visual>
-      <origin rpy="0 0 0" xyz="0 0 0.25"/>
+      <origin rpy="0 0 0" xyz="0 0 0.05" />
       <geometry>
-          <mesh filename="package://usv_sim/meshes/buoy2.dae" scale="0.5 0.5 0.5"/>
+        <mesh filename="package://usv_sim/meshes/buoy/orange.obj" scale="1 1 1" />
       </geometry>
     </visual>
     <inertial>
-      <origin rpy="0 0 0" xyz="0 0 0"/>
-      <mass value="5.0"/>
-      <inertia ixx="1" ixy="0.0" ixz="0.0" iyy="1" iyz="0" izz="1"/>
+      <origin rpy="0 0 0" xyz="0 0 0" />
+      <mass value="5.0" />
+      <inertia ixx="1" ixy="0.0" ixz="0.0" iyy="1" iyz="0" izz="1" />
     </inertial>
     <collision>
-      <origin rpy="0 0 0" xyz="0 0 0.25"/>
-     <geometry>
-          <mesh filename="package://usv_sim/meshes/buoy2.dae" scale="0.5 0.5 0.5"/>
+      <origin rpy="0 0 0" xyz="0 0 0.05" />
+      <geometry>
+        <mesh filename="package://usv_sim/meshes/buoy/orange.obj" scale="1 1 1" />
       </geometry>
     </collision>
-		<buoyancy>
-        	<compensation>10</compensation>
-          	<origin xyz="0 0 0.05"/>
-          	<limit radius="0.25"/>
-          	<windVelocity>none</windVelocity>
-          	<damping rpy="20 20 20" xyz="100 100 50"/>
-	  	  	<waterVelocity>none</waterVelocity>
-        </buoyancy>
+    <buoyancy>
+      <compensation>10</compensation>
+      <origin xyz="0 0 0.05" />
+      <limit radius="0.25" />
+      <windVelocity>none</windVelocity>
+      <damping rpy="20 20 20" xyz="100 100 50" />
+      <waterVelocity>none</waterVelocity>
+    </buoyancy>
   </link>
 </robot>

Commit message: Making buoys smaller and deleting unneeded files

File: usv_sim/xacro/buoy.xacro (robot description, xacro)
@@ -16,5 +16,5 @@
       <origin rpy="0 0 0" xyz="0 0 0.05" />
       <geometry>
-        <mesh filename="package://usv_sim/meshes/buoy/orange.obj" scale="1 1 1" />
+        <mesh filename="package://usv_sim/meshes/buoy/orange_collis.obj" scale="1 1 1" />
       </geometry>
     </collision>
